Commit message: Graph, env,
Added avg score to data and graph, blank env is no longer just blank but is rather a blank maze

File: pybullet/models/scenes/blank/blank.urdf (robot description, URDF)
Before this commit: robot blank, 1 links, 0 joints
Links:
- link base_link: geometry collision mesh filename=meshes/blank.obj scale=0.02 0.02 0.01; visual mesh filename=meshes/blank.obj scale=0.02 0.02 0.01
