Commit message: update the straight env

File: pybullet/models/scenes/straight/straight.urdf (robot description, URDF)
Before this commit: robot straight_env, 1 links, 0 joints
Links:
- link base_link: geometry collision mesh filename=meshes/straight.obj scale=0.02 0.02 0.01; visual mesh filename=meshes/straight.obj scale=0.02 0.02 0.01
